File: F3K_Battery_manager.sch (KiCad schematic (older format))
At the start: 14 parts, among them J1 Coil 1, J2 Coil 2, J3 BATT +, J4 BATT -, J5 DEBUG, J6 Serial, J7 Receiver, Q1 CSD13385F5, Q2 CSD13385F5, U1 DRV5032

Commit message: Added budget
Parts:
- added AE1: Wireless antenna, symbol Antenna_Loop
Connections:
- no-connect marks 0 -> 2
Other:
- note added: "Antenna for Kicost\n"
Changed lines of the file:
@@
 Wire Wire Line
 	1850 4450 2100 4450
+$Comp
+L Antenna_Loop AE1
+U 1 1 5AB18F00
+P 1100 4350
+F 0 "AE1" H 1150 4600 50  0000 C CNN
+F 1 "Wireless antenna" H 1150 4550 50  0000 C CNN
+F 2 "" H 1100 4350 50  0001 C CNN
+F 3 "" H 1100 4350 50  0001 C CNN
+F 4 "IWAS3827ECEB100J50" H 1100 4350 60  0001 C CNN "MPN"
+	1    1100 4350
+	0    -1   -1   0
+$EndComp
+NoConn ~ 1300 4250
+NoConn ~ 1300 4350
+Text Notes 550  3950 0    60   ~ 0
+Antenna for Kicost\n
 $EndSCHEMATC
