File: boost_converter.sch (KiCad schematic (older format))
At the start: 13 parts, among them U4 TPS61236P

Commit message: Added resistor and capacitor values, footprints and NPNs
Parts:
- C10: MPN (none) -> GRM1555C1H100FA01D
- C11: value 33uF 4V -> 33uF 6V3; footprint (none) -> Capacitors_SMD:C_0805; MPN GRM21BR60G336ME15L -> C2012X5R0J336M125AC
Changed lines of the file:
@@
 F 2 "Capacitors_SMD:C_0402" H 6588 3400 50  0001 C CNN
 F 3 "" H 6550 3550 50  0001 C CNN
+F 4 "GRM1555C1H100FA01D" H 6550 3550 60  0001 C CNN "MPN"
 	1    6550 3550
 	1    0    0    -1
@@
 $EndComp
 $Comp
-L GND #PWR37
+L GND #PWR032
 U 1 1 5AA40E28
 P 6850 4200
-F 0 "#PWR37" H 6850 3950 50  0001 C CNN
+F 0 "#PWR032" H 6850 3950 50  0001 C CNN
 F 1 "GND" H 6850 4050 50  0000 C CNN
 F 2 "" H 6850 4200 50  0001 C CNN
@@
 $EndComp
 $Comp
-L GND #PWR36
+L GND #PWR033
 U 1 1 5AA40E49
 P 5850 4550
-F 0 "#PWR36" H 5850 4300 50  0001 C CNN
+F 0 "#PWR033" H 5850 4300 50  0001 C CNN
 F 1 "GND" H 5850 4400 50  0000 C CNN
 F 2 "" H 5850 4550 50  0001 C CNN
@@
 P 9300 3800
 F 0 "C11" H 9325 3900 50  0000 L CNN
-F 1 "33uF 4V" H 9350 3700 50  0000 L CNN
-F 2 "" H 9338 3650 50  0001 C CNN
+F 1 "33uF 6V3" H 9350 3700 50  0000 L CNN
+F 2 "Capacitors_SMD:C_0805" H 9338 3650 50  0001 C CNN
 F 3 "" H 9300 3800 50  0001 C CNN
-F 4 "GRM21BR60G336ME15L" H 9300 3800 60  0001 C CNN "MPN"
+F 4 "C2012X5R0J336M125AC" H 9300 3800 60  0001 C CNN "MPN"
 	1    9300 3800
 	1    0    0    -1
 $EndComp
 $Comp
-L GND #PWR39
+L GND #PWR034
 U 1 1 5AA40FE1
 P 9300 4200
-F 0 "#PWR39" H 9300 3950 50  0001 C CNN
+F 0 "#PWR034" H 9300 3950 50  0001 C CNN
 F 1 "GND" H 9300 4050 50  0000 C CNN
 F 2 "" H 9300 4200 50  0001 C CNN
@@
 $EndComp
 $Comp
-L GND #PWR33
+L GND #PWR035
 U 1 1 5AA412DC
 P 3800 4200
-F 0 "#PWR33" H 3800 3950 50  0001 C CNN
+F 0 "#PWR035" H 3800 3950 50  0001 C CNN
 F 1 "GND" H 3800 4050 50  0000 C CNN
 F 2 "" H 3800 4200 50  0001 C CNN
@@
 ENA
 $Comp
-L +BATT #PWR32
+L +BATT #PWR036
 U 1 1 5AA423A0
 P 3650 3450
-F 0 "#PWR32" H 3650 3300 50  0001 C CNN
+F 0 "#PWR036" H 3650 3300 50  0001 C CNN
 F 1 "+BATT" H 3650 3590 50  0000 C CNN
 F 2 "" H 3650 3450 50  0001 C CNN
@@
 $EndComp
 $Comp
-L GND #PWR38
+L GND #PWR037
 U 1 1 5AB62B99
 P 8250 4200
-F 0 "#PWR38" H 8250 3950 50  0001 C CNN
+F 0 "#PWR037" H 8250 3950 50  0001 C CNN
 F 1 "GND" H 8250 4050 50  0000 C CNN
 F 2 "" H 8250 4200 50  0001 C CNN
@@
 	5050 4100 5050 4200
 $Comp
-L GND #PWR35
+L GND #PWR038
 U 1 1 5AB63392
 P 5050 4550
-F 0 "#PWR35" H 5050 4300 50  0001 C CNN
+F 0 "#PWR038" H 5050 4300 50  0001 C CNN
 F 1 "GND" H 5050 4400 50  0000 C CNN
 F 2 "" H 5050 4550 50  0001 C CNN
@@
 Connection ~ 5050 4100
 $Comp
-L GND #PWR34
+L GND #PWR039
 U 1 1 5AB634B2
 P 4850 4550
-F 0 "#PWR34" H 4850 4300 50  0001 C CNN
+F 0 "#PWR039" H 4850 4300 50  0001 C CNN
 F 1 "GND" H 4850 4400 50  0000 C CNN
 F 2 "" H 4850 4550 50  0001 C CNN
